Commit message: update urdf

File: husky_description/urdf/husky_macro.urdf.xacro (robot description, xacro)
@@ -14,7 +14,9 @@
   <xacro:arg name="urdf_extras" default="$(optenv CPR_URDF_EXTRAS empty.urdf)" />
   <xacro:arg name="serial_port" default="$(optenv HUSKY_SERIAL_PORT /dev/prolific)" />
+  <xacro:arg name="use_nominal_extrinsics" default="false" />
   <!-- Included URDF/XACRO Files -->
   <xacro:include filename="$(find husky_description)/urdf/decorations.urdf.xacro" />
   <xacro:include filename="$(find husky_description)/urdf/wheel.urdf.xacro" />
+  <xacro:include filename="$(find realsense2_description)/urdf/_d435i.urdf.xacro"/>
   <xacro:include filename="$(find husky_description)/urdf/accessories/intel_realsense.urdf.xacro"/>
   <!-- <xacro:include filename="$(find husky_description)/urdf/accessories/sick_lms1xx_mount.urdf.xacro"/> -->
@@ -90,4 +92,462 @@
       <child link="${prefix}gps_link" />
     </joint>
+  <link
+    name="plate_link">
+    <inertial>
+      <origin
+        xyz="1.51841739686117E-06 0.217702480334483 0.10337194353501"
+        rpy="0 0 0" />
+      <mass
+        value="3.43579942471049" />
+      <inertia
+        ixx="0.0839007972174073"
+        ixy="-8.16841419972499E-18"
+        ixz="-2.45268280782475E-12"
+        iyy="0.123973068418061"
+        iyz="0.000189419828769455"
+        izz="0.0421838222352592" />
+    </inertial>
+    <visual>
+      <origin
+        xyz="0 0 0"
+        rpy="0 0 0" />
+      <geometry>
+        <mesh
+          filename="package://husky_description/meshes/sensors/plate_link.STL" />
+      </geometry>
+      <material
+        name="">
+        <color
+          rgba="0.250980392156863 0.250980392156863 0.250980392156863 1" />
+      </material>
+    </visual>
+    <collision>
+      <origin
+        xyz="0 0 0"
+        rpy="0 0 0" />
+      <geometry>
+        <mesh
+          filename="package://husky_description/meshes/sensors/plate_link.STL" />
+      </geometry>
+    </collision>
+  </link>
+   <joint
+    name="plate_joint"
+    type="fixed">
+    <origin
+      xyz="0 0 0"
+      rpy="0 0 1.57" />
+    <parent
+      link="base_link" />
+    <child
+      link="plate_link" />
+    <axis
+      xyz="0 0 0" />
+  </joint>
+  <link
+    name="l_gnss_link">
+    <inertial>
+      <origin
+        xyz="0.000124609008117726 7.66617830327831E-09 0.0102528003680311"
+        rpy="0 0 0" />
+      <mass
+        value="0.0701964032409456" />
+      <inertia
+        ixx="2.17814587000315E-05"
+        ixy="2.83762091549197E-11"
+        ixz="4.22773611169793E-09"
+        iyy="2.02617157250508E-05"
+        iyz="-5.75688515653656E-12"
+        izz="3.64648240418004E-05" />
+    </inertial>
+    <visual>
+      <origin
+        xyz="0 0 0"
+        rpy="0 0 0" />
+      <geometry>
+        <mesh
+          filename="package://husky_description/meshes/sensors/l_gnss_link.STL" />
+      </geometry>
+      <material
+        name="">
+        <color
+          rgba="0.643137254901961 0.509803921568627 0 1" />
+      </material>
+    </visual>
+    <collision>
+      <origin
+        xyz="0 0 0"
+        rpy="0 0 0" />
+      <geometry>
+        <mesh
+          filename="package://husky_description/meshes/sensors/l_gnss_link.STL" />
+      </geometry>
+    </collision>
+  </link>
+  <joint
+    name="l_gnss_joint"
+    type="fixed">
+    <origin
+      xyz="0.222500000000147 -0.232687355330983 0.409425000000008"
+      rpy="0 0 3.14159265358979" />
+    <parent
+      link="plate_link" />
+    <child
+      link="l_gnss_link" />
+    <axis
+      xyz="0 0 0" />
+  </joint>
+  <link
+    name="r_gnss_link">
+    <inertial>
+      <origin
+        xyz="0.000124609008123611 7.66617838654504E-09 0.010252800368031"
+        rpy="0 0 0" />
+      <mass
+        value="0.0701964032409453" />
+      <inertia
+        ixx="2.17814587000314E-05"
+        ixy="2.83762091330025E-11"
+        ixz="4.22773611182136E-09"
+        iyy="2.02617157250507E-05"
+        iyz="-5.75688522696241E-12"
+        izz="3.64648240418002E-05" />
+    </inertial>
+    <visual>
+      <origin
+        xyz="0 0 0"
+        rpy="0 0 0" />
+      <geometry>
+        <mesh
+          filename="package://husky_description/meshes/sensors/r_gnss_link.STL" />
+      </geometry>
+      <material
+        name="">
+        <color
+          rgba="0.643137254901961 0.509803921568627 0 1" />
+      </material>
+    </visual>
+    <collision>
+      <origin
+        xyz="0 0 0"
+        rpy="0 0 0" />
+      <geometry>
+        <mesh
+          filename="package://husky_description/meshes/sensors/r_gnss_link.STL" />
+      </geometry>
+    </collision>
+  </link>
+  <joint
+    name="r_gnss_joint"
+    type="fixed">
+    <origin
+      xyz="-0.222499999999849 -0.232687355330983 0.409425000000011"
+      rpy="0 0 0" />
+    <parent
+      link="plate_link" />
+    <child
+      link="r_gnss_link" />
+    <axis
+      xyz="0 0 0" />
+  </joint>
+  <link
+    name="os_sensor">
+    <inertial>
+      <origin
+        xyz="0.00189899503220095 -2.27467289361314E-06 -0.0052562660592802"
+        rpy="0 0 0" />
+      <mass
+        value="0.818090335795892" />
+      <inertia
+        ixx="0.00109605890566487"
+        ixy="5.828824898437E-09"
+        ixz="9.14474609291753E-06"
+        iyy="0.000788817921503734"
+        iyz="-1.30836536867828E-08"
+        izz="0.00151823152143701" />
+    </inertial>
+    <visual>
+      <origin
+        xyz="0 0 0"
+        rpy="0 0.785398163397443 -1.57079632679489" />
+      <geometry>
+        <mesh
+          filename="package://husky_description/meshes/sensors/os_sensor.STL" />
+      </geometry>
+      <material
+        name="">
+        <color
+          rgba="0.792156862745098 0.819607843137255 0.933333333333333 1" />
+      </material>
+    </visual>
+    <collision>
+      <origin
+        xyz="0 0 0"
+        rpy="0 0 0" />
+      <geometry>
+        <mesh
+          filename="package://husky_description/meshes/sensors/os_sensor.STL" />
+      </geometry>
+    </collision>
+  </link>
+  <joint
+    name="ouster_joint"
+    type="fixed">
+    <origin
+      xyz="0 -0.484709604427087 0.312829328932582"
+      rpy="0 0.785398163397443 -1.57079632679489" />
+    <parent
+      link="plate_link" />
+    <child
+      link="os_sensor" />
+    <axis
+      xyz="0 0 0" />
+  </joint>
+  <link name="os_imu" />
+  <link name="os_lidar" />
+    <joint name="ouster_imu_link_joint" type="fixed">
+      <parent link="os_sensor" />
+      <child link="os_imu" />
+      <origin xyz="0.006253 -0.011775 0.007645" rpy="0 0 0" />
+    </joint>
+    <joint name="ouster_lidar_link_joint" type="fixed">
+      <parent link="os_sensor" />
+      <child link="os_lidar" />
+      <origin xyz="0.0 0.0 0.03618" rpy="0 0 3.14" />
+    </joint>
+  <link
+    name="l_rs_link">
+    <inertial>
+      <origin
+        xyz="0.00168162835091112 2.49429217691333E-06 -0.0132723219640002"
+        rpy="0 0 0" />
+      <mass
+        value="0.0381925087892179" />
+      <inertia
+        ixx="2.11195789050057E-06"
+        ixy="-7.8505168622085E-09"
+        ixz="4.52141592209166E-08"
+        iyy="2.22593860090099E-05"
+        iyz="-1.30044992733574E-08"
+        izz="2.3576234083329E-05" />
+    </inertial>
+    <visual>
+      <origin
+        xyz="0 0 0"
+        rpy="0 0 0" />
+      <geometry>
+        <mesh
+          filename="package://husky_description/meshes/sensors/l_rs_link.STL" />
+      </geometry>
+      <material
+        name="">
+        <color
+          rgba="0.792156862745098 0.819607843137255 0.933333333333333 1" />
+      </material>
+    </visual>
+    <collision>
+      <origin
+        xyz="0 0 0"
+        rpy="0 0 0" />
+      <geometry>
+        <mesh
+          filename="package://husky_description/meshes/sensors/l_rs_link.STL" />
+      </geometry>
+    </collision>
+  </link>
+  <joint
+    name="l_rs_joint"
+    type="fixed">
+    <origin
+      xyz="0.22755231806118 -0.232687355330983 0.382669786798316"
+      rpy="-1.83259571459405 0 -1.5707963267949" />
+    <parent
+      link="plate_link" />
+    <child
+      link="l_rs_link" />
+    <axis
+      xyz="0 0 0" />
+  </joint>
+  <link
+    name="r_rs_link">
+    <inertial>
+      <origin
+        xyz="0.00168164156528267 2.49000785967901E-06 -0.0132723145550583"
+        rpy="0 0 0" />
+      <mass
+        value="0.0381924678690491" />
+      <inertia
+        ixx="2.11198182723984E-06"
+        ixy="-7.84310817836137E-09"
+        ixz="4.52129507808281E-08"
+        iyy="2.22593611799269E-05"
+        iyz="-1.30036949521211E-08"
+        izz="2.35762341803649E-05" />
+    </inertial>
+    <visual>
+      <origin
+        xyz="0 0 0"
+        rpy="0 0 0" />
+      <geometry>
+        <mesh
+          filename="package://husky_description/meshes/sensors/r_rs_link.STL" />
+      </geometry>
+      <material
+        name="">
+        <color
+          rgba="0.792156862745098 0.819607843137255 0.933333333333333 1" />
+      </material>
+    </visual>
+    <collision>
+      <origin
+        xyz="0 0 0"
+        rpy="0 0 0" />
+      <geometry>
+        <mesh
+          filename="package://husky_description/meshes/sensors/r_rs_link.STL" />
+      </geometry>
+    </collision>
+  </link>
+  <joint
+    name="r_rs_joint"
+    type="fixed">
+    <origin
+      xyz="-0.227552318061205 -0.232692455331 0.382669786798291"
+      rpy="1.83259571459412 0 -1.5707963267949" />
+    <parent
+      link="plate_link" />
+    <child
+      link="r_rs_link" />
+    <axis
+      xyz="0 0 0" />
+  </joint>
+  <link
+    name="f_rs_link">
+    <inertial>
+      <origin
+        xyz="0.00168172493037785 2.49411756339524E-06 -0.0132722979188402"
+        rpy="0 0 0" />
+      <mass
+        value="0.0381925640618229" />
+      <inertia
+        ixx="2.11195644163414E-06"
+        ixy="-7.84806623029052E-09"
+        ixz="4.52136752794108E-08"
+        iyy="2.22593860722202E-05"
+        iyz="-1.30042954639318E-08"
+        izz="2.35762325846014E-05" />
+    </inertial>
+    <visual>
+      <origin
+        xyz="0 0 0"
+        rpy="0 0 0" />
+      <geometry>
+        <mesh
+          filename="package://husky_description/meshes/sensors/f_rs_link.STL" />
+      </geometry>
+      <material
+        name="">
+        <color
+          rgba="0.792156862745098 0.819607843137255 0.933333333333333 1" />
+      </material>
+    </visual>
+    <collision>
+      <origin
+        xyz="0 0 0"
+        rpy="0 0 0" />
+      <geometry>
+        <mesh
+          filename="package://husky_description/meshes/sensors/f_rs_link.STL" />
+      </geometry>
+    </collision>
+  </link>
+  <joint
+    name="f_rs_joint"
+    type="fixed">
+    <origin
+      xyz="9.96250059669459E-05 -0.510747555330992 0.163366540707293"
+      rpy="1.5707963267949 0 0" />
+    <parent
+      link="plate_link" />
+    <child
+      link="f_rs_link" />
+    <axis
+      xyz="0 0 0" />
+  </joint>
+ <!--
+  <link
+    name="ins_link">
+  </link>
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